Commit message: Config tweaks to get rtabmap working with nav2 - more or less. Some calibration is still called for (e.g. robot xacro) and rtabmap output for static scenes is ... dubious. We may need more lidars!

File: src/ugv_main/ugv_description/xacro/robot.xacro (robot description, xacro)
@@ -124,5 +124,5 @@
     <xacro:property name="battery_orin_offset" value="${battery_height/2 + orin_height/2 + velcro_height}"/>
     <xacro:property name="orin_lidar_offset" value="${orin_height/2 + lidar_height/2 + velcro_height}"/>
-    <xacro:property name="orin_d435_offset_x" value="${orin_length/2 + d435_length/2 + velcro_height}"/>
+    <xacro:property name="orin_d435_offset_x" value="${orin_length/2 + d435_length/2 + velcro_height*2}"/>
     <xacro:property name="orin_d435_offset_z" value="${orin_height/2 - d435_height/2}"/>
     <xacro:property name="orin_gps_offset_x" value=".034"/>
@@ -213,5 +213,5 @@
     <!-- camera joint -->
     <joint name="d435_joint" type="fixed">
-        <origin xyz="${orin_d435_offset_x} 0 ${orin_d435_offset_z}" rpy="0 0 0"/>
+	    <origin xyz="${orin_d435_offset_x} 0 ${orin_d435_offset_z-.02}" rpy="0 ${35.0*3.1416/180.0} 0"/>
         <parent link="orin_link"/>
         <child link="camera_link"/>
