Commit message: Add calibrated ugv.xacro file to ugv_description package. A mirror of this commit from the simulation host will follow immediately. This commit is from Orin (the robot).

File: src/ugv_main/ugv_description/xacro/ugv.xacro (robot description, xacro)
@@ -138,5 +138,5 @@
     <xacro:box_link name="orin_link" length="${orin_length}" width="${orin_width}" height="${orin_height}" density="${orin_density}" color="0.45 0.45 0.45 1.0"/>
     <xacro:box_link name="lidar_link" length="${lidar_length}" width="${lidar_width}" height="${lidar_height}" density="${lidar_density}" color="0.0 0.0 0.0 1.0"/>
-    <xacro:box_link name="camera_link" length="${d435_length}" width="${d435_width}" height="${d435_height}" density="${d435_density}" color="0.7 0.7 0.7 1.0"/>
+    <xacro:box_link name="camera_pre_link" length="${d435_length}" width="${d435_width}" height="${d435_height}" density="${d435_density}" color="0.7 0.7 0.7 1.0"/>
     <xacro:box_link name="gps_link" length="${gps_length}" width="${gps_width}" height="${gps_height}" density="${gps_density}" color="1.0 1.0 1.0 1.0"/>
     <xacro:wheel_link name="left_wheel_link" radius="${wheel_radius}" width="${wheel_width}" density="${wheel_density}" color="0.1 0.1 0.1 1.0"/>
@@ -152,4 +152,5 @@
     </link>
     <link name="camera_optical_link"/>
+    <link name="camera_link"/>
     <!-- Joints -->
     <joint name="base_footprint_joint" type="fixed">
@@ -216,4 +217,10 @@
 	    <origin xyz="${orin_d435_offset_x} 0 ${orin_d435_offset_z-.02}" rpy="0 ${35.0*3.1416/180.0} 0"/>
         <parent link="orin_link"/>
+        <child link="camera_pre_link"/>
+    </joint>
+    <!-- camera calibration joint -->
+    <joint name="d435_calibration_joint" type="fixed">
+	    <origin xyz="-0.00087293  0.00217825  0.00588482" rpy="-0.01896374  0.01090149  0.00443497"/>
+        <parent link="camera_pre_link"/>
         <child link="camera_link"/>
     </joint>

Commit message: Update xacro file after depth camera calibration.

File: src/ugv_main/ugv_description/xacro/ugv.xacro (robot description, xacro)
@@ -221,5 +221,5 @@
     <!-- camera calibration joint -->
     <joint name="d435_calibration_joint" type="fixed">
-	    <origin xyz="-0.00087293  0.00217825  0.00588482" rpy="-0.01896374  0.01090149  0.00443497"/>
+	    <origin xyz="0.00185596  0.00479639 -0.00043884" rpy="0.00352776  0.01112985 -0.00777017"/>
         <parent link="camera_pre_link"/>
         <child link="camera_link"/>

Commit message: Updates to support new sensor fusion/code fusion via ugv_main/ugv. Beginnings of updates to ugv_main/ugv/launch - mostly copied from ugv_main/ugv_bringup/launch. This should support on-robot lidar/depth camera calibration.

File: src/ugv_main/ugv_description/xacro/ugv.xacro (robot description, xacro)
@@ -137,5 +137,5 @@
     <xacro:box_link name="battery_link" length="${battery_length}" width="${battery_width}" height="${battery_height}" density="${battery_density}" color="0.25 0.25 0.25 1.0"/>
     <xacro:box_link name="orin_link" length="${orin_length}" width="${orin_width}" height="${orin_height}" density="${orin_density}" color="0.45 0.45 0.45 1.0"/>
-    <xacro:box_link name="lidar_link" length="${lidar_length}" width="${lidar_width}" height="${lidar_height}" density="${lidar_density}" color="0.0 0.0 0.0 1.0"/>
+    <xacro:box_link name="lidar_pre_link" length="${lidar_length}" width="${lidar_width}" height="${lidar_height}" density="${lidar_density}" color="0.0 0.0 0.0 1.0"/>
     <xacro:box_link name="camera_pre_link" length="${d435_length}" width="${d435_width}" height="${d435_height}" density="${d435_density}" color="0.7 0.7 0.7 1.0"/>
     <xacro:box_link name="gps_link" length="${gps_length}" width="${gps_width}" height="${gps_height}" density="${gps_density}" color="1.0 1.0 1.0 1.0"/>
@@ -153,4 +153,5 @@
     <link name="camera_optical_link"/>
     <link name="camera_link"/>
+    <link name="lidar_link"/>
     <!-- Joints -->
     <joint name="base_footprint_joint" type="fixed">
@@ -211,4 +212,10 @@
         <origin xyz="-.045 0 ${orin_lidar_offset}" rpy="0 0 0"/>
         <parent link="orin_link"/>
+        <child link="lidar_pre_link"/>
+    </joint>
+    <!-- lidar calibration joint -->
+    <joint name="lidar_calibration_joint" type="fixed">
+	    <origin xyz="0 0 0" rpy="0 0 0"/>
+        <parent link="lidar_pre_link"/>
         <child link="lidar_link"/>
     </joint>
